File: Electrical Files/H&S Module/MC Control.kicad_sch (KiCad schematic)
At the start: 2 parts, among them J7 PPTC151LFBN-RC, J8 PPTC151LFBN-RC

Commit message: Control Hub, Flexible Hotplate, Housing Fan
Parts:
- added C1, C5, C6: 0.1u, Capacitor_SMD:C_0603_1608Metric_Pad1.08x0.95mm_HandSolder, symbol Device:C
- added J5: 1.27mm pin header, Connector_PinHeader_1.27mm:PinHeader_1x02_P1.27mm_Vertical, symbol Connector:Conn_01x02_Pin
- added J9: Conn_01x02, Connector_Molex:Molex_Mini-Fit_Jr_5569-02A2_2x01_P4.20mm_Horizontal, symbol Connector_Generic:Conn_01x02
- added M1: Fan, Connector_JST:JST_PH_B2B-PH-K_1x02_P2.00mm_Vertical, symbol Motor:Fan
- added Q9: BSS138, Package_TO_SOT_SMD:SOT-23-3, symbol Simulation_SPICE:NMOS
- added R15: 2k, Resistor_SMD:R_0603_1608Metric_Pad0.98x0.95mm_HandSolder, symbol Device:R
- added R16: 10k, Resistor_SMD:R_0603_1608Metric_Pad0.98x0.95mm_HandSolder, symbol Device:R
- added R2: 120, Resistor_SMD:R_0603_1608Metric_Pad0.98x0.95mm_HandSolder, symbol Device:R
- added TH1: Thermistor_US, Resistor_SMD:R_0603_1608Metric_Pad0.98x0.95mm_HandSolder, symbol Device:Thermistor_US
- added U7: MCP2562-E-SN, Package_SO:SOIC-8_3.9x4.9mm_P1.27mm, symbol Interface_CAN_LIN:MCP2562-E-SN
Connections:
- net +3.3V: now also C1.1, C6.1, M1.1 (+), TH1.1, U7.5 (Vio)
- net +5V: now also C5.2, U7.3 (VDD)
- net GND: now also C1.2, C5.1, C6.2, Q9.3 (S), R15.2, R16.1, U7.2 (VSS), U7.8 (STBY)
- net Motor_4: now also J8.9 (Pin_9); no longer J7.13 (Pin_13)
- net TX/RX+: now reaches J7.5 (Pin_5)
- net TX/RX+: now also U7.1 (TXD)
- net at J8.5 (Pin_5): now also Q9.2 (G), R15.1
- net at J8.6 (Pin_6): now also R16.2, TH1.2
- new net: M1.2 (-), Q9.1 (D)
- new net: J5.2 (Pin_2), R2.2
- new net CAN+: J9.1 (Pin_1), R2.1, U7.7 (CANH)
- new net CAN-: J5.1 (Pin_1), J9.2 (Pin_2), U7.6 (CANL)
- new net TX/RX-: J7.13 (Pin_13), U7.4 (RXD)
Other:
- note added: "1 Can OUT"
- note added: "3 or 4 power out"
- note added: "CANBUS Daisy Chain?"
- note added: "Filtering?"
- note added: "High pass flters on inputs/outpute?"
- note added: "How to protect PWM signals from EMI?"
- note added: "Toggle terminating resistors"
- note added: "Verify Pinouts"
