File: Electrical Files/H&S Module/Motor Array.kicad_sch (KiCad schematic)
At the start: 24 parts, among them M13 PPN7PA12C1, M14 PPN7PA12C1, M15 PPN7PA12C1, M16 PPN7PA12C1, M17 PPN7PA12C1, M18 PPN7PA12C1, M19 PPN7PA12C1, M20 PPN7PA12C1, M21 PPN7PA12C1, M22 PPN7PA12C1, M23 PPN7PA12C1, M24 PPN7PA12C1, Q1 BSR802NL6327HTSA1, Q2 BSR802NL6327HTSA1, Q3 BSR802NL6327HTSA1, Q8 BSR802NL6327HTSA1

Commit message: Control Hub, Flexible Hotplate, Housing Fan
Parts:
- D1, D2, D3, D4: footprint (none) -> Diode_SMD:D_SOD-323
Other:
- note added: "Select diodes"
Changed lines of the file:
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@@
 	(generator_version "10.0")
 	(paper "A4")
+	(text "Select diodes"
+		(exclude_from_sim no)
+		(at 161.29 33.274 0)
+		(effects
+			(font
+				(size 1.27 1.27)
+			)
+		)
+	)
 	(junction
 		(at 121.92 54.61)
@@
 			)
 		)
-		(property "Footprint" ""
+		(property "Footprint" "Diode_SMD:D_SOD-323"
 			(at 115.57 43.18 0)
 			(hide yes)
@@
 			)
 		)
-		(property "Footprint" ""
+		(property "Footprint" "Diode_SMD:D_SOD-323"
 			(at 82.55 43.18 0)
 			(hide yes)
@@
 			)
 		)
-		(property "Footprint" ""
+		(property "Footprint" "Diode_SMD:D_SOD-323"
 			(at 148.59 43.18 0)
 			(hide yes)
@@
 			)
 		)
-		(property "Footprint" ""
+		(property "Footprint" "Diode_SMD:D_SOD-323"
 			(at 48.26 44.45 0)
 			(hide yes)
