File: Electrical Files/H&S Module/S&H Management board.kicad_pcb (KiCad board)
At the start: 4 copper layers, 119.4 x 77.2 mm, 57 parts, among them J1 DF11-4DP-2DSA(24), J2 DF11-4DP-2DSA(24), J3 DF11-4DP-2DSA(24), J4 DF11-4DP-2DSA(24), J7 PPTC151LFBN-RC, J8 PPTC151LFBN-RC, M13 PPN7PA12C1, M14 PPN7PA12C1, M15 PPN7PA12C1, M16 PPN7PA12C1, M17 PPN7PA12C1, M18 PPN7PA12C1, M19 PPN7PA12C1, M20 PPN7PA12C1, M21 PPN7PA12C1, M22 PPN7PA12C1, M23 PPN7PA12C1, M24 PPN7PA12C1, Q1 BSR802NL6327HTSA1, Q2 BSR802NL6327HTSA1, Q3 BSR802NL6327HTSA1, Q4 IRLML6344TRPBF, Q5 IRLML6344TRPBF, Q6 IRLML6344TRPBF, Q7 IRLML6344TRPBF, Q8 BSR802NL6327HTSA1, U1 TPS54560BDDA

Commit message: Control Hub, Flexible Hotplate, Housing Fan
Parts:
- added C1: 0.1u, Capacitor_SMD:C_0603_1608Metric_Pad1.08x0.95mm_HandSolder, F.Cu at (140.2, 57.8)
- added C10: 100uF, Capacitor_SMD:C_0603_1608Metric_Pad1.08x0.95mm_HandSolder, F.Cu at (141.3, 62.1)
- added C3: 10uF, Capacitor_SMD:C_0603_1608Metric_Pad1.08x0.95mm_HandSolder, F.Cu at (141.3, 66.8)
- added C4: 10uF, Capacitor_SMD:C_0603_1608Metric_Pad1.08x0.95mm_HandSolder, F.Cu at (141.3, 65.2)
- added C5: 0.1u, Capacitor_SMD:C_0603_1608Metric_Pad1.08x0.95mm_HandSolder, F.Cu at (136.5, 63.8)
- added C6: 0.1u, Capacitor_SMD:C_0603_1608Metric_Pad1.08x0.95mm_HandSolder, F.Cu at (161.6, 59.0)
- added C9: 100uF, Capacitor_SMD:C_0603_1608Metric_Pad1.08x0.95mm_HandSolder, F.Cu at (141.3, 63.6)
- added D1: D_Schottky, Diode_SMD:D_SOD-323, F.Cu at (106.0, 80.5)
- added D10: PESD3V3L1BA, Diode_SMD:D_SOD-323F, F.Cu at (154.1, 89.0)
- added D2: D_Schottky, Diode_SMD:D_SOD-323, F.Cu at (109.3, 77.7)
- added D3: D_Schottky, Diode_SMD:D_SOD-323, F.Cu at (169.7, 76.3)
- added D4: D_Schottky, Diode_SMD:D_SOD-323, F.Cu at (172.7, 73.4)
- added D5: PESD3V3L1BA, Diode_SMD:D_SOD-323F, F.Cu at (124.5, 89.3)
- added D8: PESD3V3L1BA, Diode_SMD:D_SOD-323F, F.Cu at (122.4, 90.3)
- added D9: PESD3V3L1BA, Diode_SMD:D_SOD-323F, F.Cu at (156.1, 90.5)
- added J6: Conn_01x02, Connector_Molex:Molex_Mini-Fit_Jr_5569-02A2_2x01_P4.20mm_Horizontal, F.Cu at (142.5, 46.3)
- added J9: Conn_01x02, Connector_Molex:Molex_Mini-Fit_Jr_5569-02A2_2x01_P4.20mm_Horizontal, F.Cu at (136.0, 46.3)
- added M1: Fan, Connector_JST:JST_PH_B2B-PH-K_1x02_P2.00mm_Vertical, F.Cu at (158.2, 58.1)
- added Q9: BSS138, Package_TO_SOT_SMD:SOT-23-3, F.Cu at (152.8, 59.1)
- added R15: 2k, Resistor_SMD:R_0603_1608Metric_Pad0.98x0.95mm_HandSolder, F.Cu at (152.8, 56.4)
- added R16: 10k, Resistor_SMD:R_0603_1608Metric_Pad0.98x0.95mm_HandSolder, F.Cu at (149.4, 58.3)
- added TH1: Thermistor_US, Resistor_SMD:R_0603_1608Metric_Pad0.98x0.95mm_HandSolder, F.Cu at (149.4, 55.0)
- added U7: MCP2562-E-SN, Package_SO:SOIC-8_3.9x4.9mm_P1.27mm, F.Cu at (136.6, 59.2)
- moved R8 9.85 mm to (144.2, 76.5), turned to -90 degrees
- moved R14 8.88 mm to (144.2, 62.0), turned to 90 degrees
- moved R10 8.73 mm to (144.3, 72.2), turned to 90 degrees
- moved R12 8.36 mm to (134.4, 69.6), turned to 90 degrees
- moved J7 6.56 mm to (131.6, 47.7)
- moved J8 6.56 mm to (146.9, 47.7)
- moved D7 2.80 mm to (134.8, 94.2)
- moved C17 2.52 mm to (142.9, 88.2)
- moved C18 2.52 mm to (142.9, 89.7)
- moved C19 2.52 mm to (142.9, 91.3)
- moved L1 2.52 mm to (142.1, 96.6)
Connections:
- J7 pad 13: /MC Control/Motor_4 -> /MC Control/TX/RX-
- J7 pad 5: unconnected-(J7-Pin_5-Pad5) -> /MC Control/TX/RX+
- J8 pad 5: unconnected-(J8-Pin_5-Pad5) -> Net-(J8-Pin_5)
- J8 pad 6: unconnected-(J8-Pin_6-Pad6) -> Net-(J8-Pin_6)
- J8 pad 9: unconnected-(J8-Pin_9-Pad9) -> /MC Control/Motor_4
Routing:
- net +3.3V: track 0.00 -> 65.2 mm, vias 0 -> 4
- net /MC Control/Motor_4: track 2.19 -> 51.5 mm, vias 0 -> 1
- net /Hotplates/Heat_EN4: track 1.99 -> 46.1 mm, vias 0 -> 1
- net +5V: track 51.9 -> 95.1 mm, vias 15 -> 19
- net /Hotplates/Heat_EN1: track 1.95 -> 44.0 mm, vias 0 -> 1
- net /MC Control/Motor_3: track 1.75 -> 38.2 mm
- net /MC Control/Motor_1: track 1.80 -> 33.6 mm, vias 0 -> 3
- net /Hotplates/Heat_EN2: track 1.72 -> 31.3 mm
- net /Hotplates/Heat_EN3: track 1.76 -> 28.5 mm
- net /MC Control/TX/RX-: track 0.00 -> 21.2 mm
- net /MC Control/Motor_2: track 1.83 -> 20.3 mm
- net GND: track 37.8 -> 53.6 mm, vias 25 -> 37
- net /MC Control/CAN-: track 0.00 -> 12.1 mm
- net /MC Control/CAN+: track 0.00 -> 12.0 mm
- net /Hotplates/Temp_A4: track 62.2 -> 73.8 mm
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Other:
- board size 119.4 x 77.2 mm -> 78.2 x 77.2 mm
