File: Electrical Files/H&S Module/S&H Management board.kicad_pcb (KiCad board)
At the start: 4 copper layers, 78.2 x 77.2 mm, 80 parts, among them J1 DF11-4DP-2DSA(24), J2 DF11-4DP-2DSA(24), J3 DF11-4DP-2DSA(24), J4 DF11-4DP-2DSA(24), J6 Conn_01x02, J7 PPTC151LFBN-RC, J8 PPTC151LFBN-RC, J9 Conn_01x02, M1 Fan, M13 PPN7PA12C1, M14 PPN7PA12C1, M15 PPN7PA12C1, M16 PPN7PA12C1, M17 PPN7PA12C1, M18 PPN7PA12C1, M19 PPN7PA12C1, M20 PPN7PA12C1, M21 PPN7PA12C1, M22 PPN7PA12C1, M23 PPN7PA12C1, M24 PPN7PA12C1, Q1 BSR802NL6327HTSA1, Q2 BSR802NL6327HTSA1, Q3 BSR802NL6327HTSA1, Q4 IRLML6344TRPBF, Q5 IRLML6344TRPBF, Q6 IRLML6344TRPBF, Q7 IRLML6344TRPBF, Q8 BSR802NL6327HTSA1, Q9 BSS138, U1 TPS54560BDDA, U7 MCP2562-E-SN

Commit message: New motor
Parts:
- removed M14, M15, M16, M17, M18, M19, M20, M21, M22, M23, M24: PPN7PA12C1, Gnome Foot Library:01x02 Jumper Pads
- added J5: 1.27mm pin header, Connector_PinHeader_1.27mm:PinHeader_1x02_P1.27mm_Vertical, F.Cu at (31.2, 84.4)
- added M10: GA12-N20, Pozzo Lab:GA12-N20, F.Cu at (34.8, 71.6)
- added M11: GA12-N20, Pozzo Lab:GA12-N20, F.Cu at (46.0, 71.6)
- added M12: GA12-N20, Pozzo Lab:GA12-N20, F.Cu at (57.3, 71.6)
- added M2: GA12-N20, Pozzo Lab:GA12-N20, F.Cu at (34.8, 45.1)
- added M3: GA12-N20, Pozzo Lab:GA12-N20, F.Cu at (46.0, 45.1)
- added M4: GA12-N20, Pozzo Lab:GA12-N20, F.Cu at (57.3, 45.1)
- added M5: GA12-N20, Pozzo Lab:GA12-N20, F.Cu at (68.5, 45.1)
- added M6: GA12-N20, Pozzo Lab:GA12-N20, F.Cu at (34.8, 58.4)
- added M7: GA12-N20, Pozzo Lab:GA12-N20, F.Cu at (46.0, 58.4)
- added M8: GA12-N20, Pozzo Lab:GA12-N20, F.Cu at (57.3, 58.4)
- added M9: GA12-N20, Pozzo Lab:GA12-N20, F.Cu at (68.5, 58.4)
- added R2: 120, Resistor_SMD:R_0603_1608Metric_Pad0.98x0.95mm_HandSolder, F.Cu at (31.4, 81.5)
- M13: value PPN7PA12C1 -> GA12-N20; footprint Gnome Foot Library:01x02 Jumper Pads -> Pozzo Lab:GA12-N20
Connections:
- M13 pad 2: Net-(D1-A) -> Net-(D4-A)
