File: Electrical Files/H&S Module/S&H Management board.kicad_sch (KiCad schematic)
At the start: 0 parts

Commit message: Control Hub, Flexible Hotplate, Housing Fan
Parts:
- added D10, D5, D8, D9: PESD3V3L1BA, Diode_SMD:D_SOD-323F, symbol Device:D_TVS
Connections:
- net Hotplates/Temp_A1: now also D5.1 (A1)
- net Hotplates/Temp_A2: now also D8.1 (A1)
- net Hotplates/Temp_A3: now also D9.1 (A1)
- net Hotplates/Temp_A4: now also D10.1 (A1)
- new net GND: D10.2 (A2), D5.2 (A2), D8.2 (A2), D9.2 (A2)
Other:
- note added: "SWAP with BAT54S?"
- note added: "TVS to 3P3?"
