File: Electrical Files/H&S Module/powerpath.kicad_sch (KiCad schematic)
At the start: 25 parts, among them J9 1586042-4, U1 TPS54560BDDA

Commit message: Control Hub, Flexible Hotplate, Housing Fan
Parts:
- removed D6: D_Schottky, symbol Device:D_Schottky
- removed J9: 1586042-4, symbol Connector_Generic:Conn_02x02_Counter_Clockwise
- added J6: Conn_01x02, Connector_Molex:Molex_Mini-Fit_Jr_5569-02A2_2x01_P4.20mm_Horizontal, symbol Connector_Generic:Conn_01x02
- C10, C3, C4, C9: footprint (none) -> Capacitor_SMD:C_0603_1608Metric_Pad1.08x0.95mm_HandSolder
Connections:
- net +24V: now also J6.1 (Pin_1)
- net GND: now also J6.2 (Pin_2)
