File: Electrical Files/PS Control Hub/PS Control Hub/mcControl.kicad_sch (KiCad schematic)
At the start: 4 parts, among them U1 STM32H533RETx, U2 AP2112K-3.3

Commit message: Control Hub, Flexible Hotplate, Housing Fan
Parts:
- removed U1: STM32H533RETx, Package_QFP:LQFP-64_10x10mm_P0.5mm, symbol MCU_ST_STM32H5:STM32H533RETx
- removed U2: AP2112K-3.3, Package_TO_SOT_SMD:SOT-23-5, symbol Regulator_Linear:AP2112K-3.3
- added J16, J17: PPPC192LFBN-RC, Pozzo Lab:PinSocket_2x19_P2.54mm_Vertical, symbol Connector_Generic:Conn_02x19_Odd_Even
- added U1: RBT05W24S3V3, Solar Car '25-'26:RBT10W24S05_XPP_XPR, symbol Solar Car 26:RBT05W24S05
- C1: value 10uF -> 10u; footprint (none) -> Capacitor_SMD:C_0805_2012Metric_Pad1.18x1.45mm_HandSolder
- C2: value 100uF -> 10u; footprint (none) -> Capacitor_SMD:C_0805_2012Metric_Pad1.18x1.45mm_HandSolder
Connections:
- net +5V is gone; now on net +3.3V: C2.1
- net +3.3V: now also J16.12 (Pin_12), J16.16 (Pin_16), J16.24 (Pin_24), J17.7 (Pin_7), U1.3; no longer C1.1
- net Button_1: now also J17.6 (Pin_6)
- net Chip Select: now also J17.17 (Pin_17)
- net Data/Command: now also J17.15 (Pin_15)
- net GND: now also J16.19 (Pin_19), J16.20 (Pin_20), J16.22 (Pin_22), J16.8 (Pin_8), J17.20 (Pin_20), J17.32 (Pin_32), J17.9 (Pin_9), U1.2
- net MISO: now also J17.13 (Pin_13)
- net Reset: now also J17.19 (Pin_19)
- net Rotary_A: now also J16.25 (Pin_25)
- net Rotary_B: now also J16.23 (Pin_23)
- net Rotary_Switch: now also J16.21 (Pin_21)
- net SCL: now also J17.35 (Pin_35)
- net SCLK: now also J17.36 (Pin_36)
- net SDA: now also J17.37 (Pin_37)
- net UART_RX: now also J16.30 (Pin_30)
- net UART_TX: now also J16.28 (Pin_28)
- net USB_DM: now also J17.14 (Pin_14)
- net USB_DP: now also J17.12 (Pin_12)
- new net +24V: C1.1, U1.1
Other:
- note added: "CN10"
- note added: "CN7"
- note added: "Double check pinouts"
