File: Electrical Files/PS Control Hub/PS Control Hub/powerManagement.kicad_sch (KiCad schematic)
At the start: 4 parts, among them J13 IEC_60320_C14_Receptacle

Commit message: Control Hub, Flexible Hotplate, Housing Fan
Parts:
- removed FB1, FB2: FerriteBead, symbol Device:FerriteBead
- added J3: 1017503, Pozzo Lab:CONN_1017491, symbol Connector:Screw_Terminal_01x02
- U3: value ~ -> (none)
Connections:
- net GND: now also J13.3 (PE), U3.3 (FG), U3.4 (GND), U3.5 (GND), U3.6 (GND), J3.1 (Pin_1), J3.2 (Pin_1)
- net +24V: now reaches U3.7 (+5V), U3.8 (+5V), U3.9 (+5V)
- net +24V: now also J3.3 (Pin_2), J3.4 (Pin_2)
Other:
- note added: "Change to 24V"
