File: Electrical Files/PS Control Hub/PS Control Hub/userInterface.kicad_sch (KiCad schematic)
At the start: 15 parts, among them J14 Conn_01x02, J15 Conn_01x12, P1 USB_C_Plug_USB2.0, SW1 SW_Push, SW2 SW_SPST_LED, SW3 RotaryEncoder_Switch

Commit message: Control Hub, Flexible Hotplate, Housing Fan
Parts:
- removed P1: USB_C_Plug_USB2.0, symbol Connector:USB_C_Plug_USB2.0
- removed R3, R4: 22, symbol Device:R
- removed R5: 1.5K, symbol Device:R
- removed R6: 5.1k, symbol Device:R
- removed R7: 100k, symbol Device:R
- J14: footprint (none) -> Connector_Molex:Molex_Mini-Fit_Jr_5566-02A_2x01_P4.20mm_Vertical
- J15: value Conn_01x12 -> FH12-12S-0.5SH55; symbol Connector_Generic:Conn_01x12 -> Connector_Generic:Conn_01x14
- R10, R8, R9: footprint (none) -> Resistor_SMD:R_0805_2012Metric_Pad1.20x1.40mm_HandSolder
- R11: value R -> 330; footprint (none) -> Resistor_SMD:R_0805_2012Metric_Pad1.20x1.40mm_HandSolder
- SW1: footprint (none) -> Connector_JST:JST_PH_B2B-PH-K_1x02_P2.00mm_Vertical
- SW2: footprint (none) -> Connector_JST:JST_PH_B4B-PH-K_1x04_P2.00mm_Vertical
- SW3: footprint (none) -> Connector_JST:JST_PH_B5B-PH-K_1x05_P2.00mm_Vertical
Connections:
- net +3.3V: now also SW3.4 (S1); no longer SW3.S1
- net GND: now also J15.13 (Pin_13), J15.14 (Pin_14), SW3.3 (C); no longer SW3.C
- net Rotary_A: now also SW3.1 (A); no longer SW3.A
- net Rotary_B: now also SW3.2 (B); no longer SW3.B
- net Rotary_Switch: now also SW3.5 (S2); no longer SW3.S2
Other:
- note added: "Switch to software control with hardware priority"
- note added: "Using built in user usb function"
- note removed: "VBUS Sensing?"
